Commit message: fix:根据gazebo的仿真要求删除电机属性和修改joint和Link的名字相同的问题

File: src/robot_model_pkg/biped_s4/urdf/biped_s4.urdf (robot description, URDF)
Before this commit: robot biped_s4, 61 links, 60 joints
Joints:
- removed joint head_pitch
- removed joint head_yaw
- removed joint l_arm_pitch
- removed joint l_arm_roll
- removed joint l_arm_yaw
- removed joint l_foot_pitch
- removed joint l_foot_roll
- removed joint l_forearm_pitch
- removed joint l_hand_pitch
- removed joint l_hand_roll
- removed joint l_hand_yaw
- removed joint l_index_distal_finger
- removed joint l_index_proximal_finger
- removed joint l_knee
- removed joint l_l_bar
- removed joint l_l_tendon
- removed joint l_leg_pitch
- removed joint l_leg_roll
- removed joint l_leg_yaw
- removed joint l_middle_distal_finger
- removed joint l_middle_proximal_finger
- removed joint l_pinky_distal_finger
- removed joint l_pinky_proximal_finger
- removed joint l_r_bar
- removed joint l_r_tendon
- removed joint l_ring_distal_finger
- removed joint l_ring_proximal_finger
- removed joint l_thumb_distal_pitch
- removed joint l_thumb_proximal_yaw
- removed joint r_arm_pitch
- removed joint r_arm_roll
- removed joint r_arm_yaw
- removed joint r_foot_pitch
- removed joint r_foot_roll
- removed joint r_forearm_pitch
- removed joint r_hand_pitch
- removed joint r_hand_roll
- removed joint r_hand_yaw
- removed joint r_index_distal_finger
- removed joint r_index_proximal_finger
- removed joint r_knee
- removed joint r_l_bar
- removed joint r_l_tendon
- removed joint r_leg_pitch
- removed joint r_leg_roll
- removed joint r_leg_yaw
- removed joint r_middle_distal_finger
- removed joint r_middle_proximal_finger
- removed joint r_pinky_distal_finger
- removed joint r_pinky_proximal_finger
- removed joint r_r_bar
- removed joint r_r_tendon
- removed joint r_ring_distal_finger
- removed joint r_ring_proximal_finger
- removed joint r_thumb_distal_pitch
- removed joint r_thumb_proximal_yaw
- added joint head_pitch_joint: type continuous, parent head_yaw, child head_pitch, origin xyz=0 0 0 rpy=0 0 0, axis 0 1 0
- added joint head_yaw_joint: type continuous, parent torso, child head_yaw, origin xyz=-0.0175475823124929 0 0.499400000000373 rpy=0 0 0, axis 0 0 -1
- added joint l_arm_pitch_joint: type revolute, parent torso, child l_arm_pitch, origin xyz=-0.0175475823124921 0.254700000000031 0.324500000000024 rpy=0 0 0, axis 0 1 0, limit lower=-3.14159 upper=0.523599 effort=20 velocity=1
- added joint l_arm_roll_joint: type revolute, parent l_arm_pitch, child l_arm_roll, origin xyz=0 0 0 rpy=0 0 0, axis 1 0 0, limit lower=-0.349066 upper=2.0944 effort=20 velocity=1
- added joint l_arm_yaw_joint: type revolute, parent l_arm_roll, child l_arm_yaw, origin xyz=0 0 0 rpy=0 0 0, axis 0 0 1, limit lower=-1.5708 upper=1.5708 effort=20 velocity=1
- added joint l_foot_pitch_joint: type continuous, parent l_knee, child l_foot_pitch, origin xyz=0 0 -0.346000000000004 rpy=0 0 0, axis 0 1 0
- added joint l_foot_roll_joint: type continuous, parent l_foot_pitch, child l_foot_roll, origin xyz=0 0 0 rpy=0 0 0, axis -1 0 0
- added joint l_forearm_pitch_joint: type revolute, parent l_arm_yaw, child l_forearm_pitch, origin xyz=0 0 -0.163599999999996 rpy=0 0 0, axis 0 1 0, limit lower=-1.5708 upper=0 effort=20 velocity=1
- added joint l_hand_pitch_joint: type revolute, parent l_hand_yaw, child l_hand_pitch, origin xyz=0 0 0 rpy=0 0 0, axis 0 1 0, limit lower=-1.5708 upper=1.5708 effort=20 velocity=1
- added joint l_hand_roll_joint: type revolute, parent l_hand_pitch, child l_hand_roll, origin xyz=0 0 -0.058999997180792 rpy=0 0 0, axis 1 0 0, limit lower=-1.5708 upper=1.5708 effort=20 velocity=1
- added joint l_hand_yaw_joint: type revolute, parent l_forearm_pitch, child l_hand_yaw, origin xyz=0 0 -0.132050000118071 rpy=0 0 0, axis 0 0 1, limit lower=-1.5708 upper=1.5708 effort=20 velocity=1
- added joint l_index_distal_finger_joint: type continuous, parent l_index_proximal_finger, child l_index_distal_finger, origin xyz=0.00013351949359549 0.00243998929947531 -0.0349145904281216 rpy=0 0 0, axis 0.998506141360648 -0.0546395979585221 0
- added joint l_index_proximal_finger_joint: type continuous, parent l_hand_roll, child l_index_proximal_finger, origin xyz=0.0295025377507617 0.0039487923396046 -0.174730558860478 rpy=0 -0.0311675978215656 0, axis -0.998506141360648 0.0546395979585239 0
- added joint l_knee_joint: type continuous, parent l_leg_pitch, child l_knee, origin xyz=-0.010390161952608 0 -0.249783995753446 rpy=0 0 0, axis 0 1 0
- added joint l_l_bar_joint: type continuous, parent l_knee, child l_l_bar, origin xyz=0 0.0260000000000038 -0.09 rpy=0 0 0, axis 0 1 0
- added joint l_l_tendon_joint: type continuous, parent l_l_bar, child l_l_tendon, origin xyz=-0.0579999994738184 0 0 rpy=0 0 0, axis 0 -1 0
- added joint l_leg_pitch_joint: type continuous, parent l_leg_yaw, child l_leg_pitch, origin xyz=0 0.025450000000002 -0.123449999999999 rpy=0 0 0, axis 0 1 0
- added joint l_leg_roll_joint: type continuous, parent torso, child l_leg_roll, origin xyz=-0.00254758231249262 0.0869999999999998 -0.0660000000049238 rpy=0 0 0, axis -1 0 0
- added joint l_leg_yaw_joint: type continuous, parent l_leg_roll, child l_leg_yaw, origin xyz=0 0 0 rpy=0 0 0, axis 0 0 1
- added joint l_middle_distal_finger_joint: type continuous, parent l_middle_proximal_finger, child l_middle_distal_finger, origin xyz=0 0.00292977189725752 -0.0418976901109154 rpy=0 0 0, axis 1 0 0
- added joint l_middle_proximal_finger_joint: type continuous, parent l_hand_roll, child l_middle_proximal_finger, origin xyz=0.00850000275976636 0.00820381922686209 -0.178435376742696 rpy=0 0 0, axis -1 0 0
- added joint l_pinky_distal_finger_joint: type continuous, parent l_pinky_proximal_finger, child l_pinky_distal_finger, origin xyz=-0.000139217094110203 0.00243552926671115 -0.0349148795758059 rpy=0 0 0, axis 0.998370307122341 0.0570677654761637 0
- added joint l_pinky_proximal_finger_joint: type continuous, parent l_hand_roll, child l_pinky_proximal_finger, origin xyz=-0.0332309186593585 0.00363387338808113 -0.170227008036839 rpy=0 0.0659957839625552 0, axis -0.998370307122329 -0.0570677654763681 0
- added joint l_r_bar_joint: type continuous, parent l_knee, child l_r_bar, origin xyz=0 -0.0259999999999997 -0.153 rpy=0 0 0, axis 0 1 0
- added joint l_r_tendon_joint: type continuous, parent l_r_bar, child l_r_tendon, origin xyz=-0.0579999990742142 0 -1.03629629222279E-05 rpy=0 0 0, axis 0 1 0
- added joint l_ring_distal_finger_joint: type continuous, parent l_ring_proximal_finger, child l_ring_distal_finger, origin xyz=-0.000160223392310654 0.0029279871592986 -0.0418975085137674 rpy=0 0 0, axis 0.998506141360637 0.0546395979587272 0
- added joint l_ring_proximal_finger_joint: type continuous, parent l_hand_roll, child l_ring_proximal_finger, origin xyz=-0.0126025322312212 0.0080785614881318 -0.176446661066021 rpy=0 0.0311675978215913 0, axis -0.998506141360648 -0.0546395979585319 0
- added joint l_thumb_distal_pitch_joint: type continuous, parent l_thumb_proximal_yaw, child l_thumb_distal_pitch, origin xyz=0.0120000000000023 -0.00649999999999773 0 rpy=0 0 0, axis 0 1 0
- added joint l_thumb_proximal_yaw_joint: type continuous, parent l_hand_roll, child l_thumb_proximal_yaw, origin xyz=0.0250000027597683 -0.0216278329431251 -0.110700000402975 rpy=0 0 0, axis 0 0 -1
- added joint r_arm_pitch_joint: type revolute, parent torso, child r_arm_pitch, origin xyz=-0.0175475823119764 -0.254700000000003 0.324500000000024 rpy=0 0 0, axis 0 1 0, limit lower=-3.14159 upper=0.523599 effort=20 velocity=1
- added joint r_arm_roll_joint: type revolute, parent r_arm_pitch, child r_arm_roll, origin xyz=0 0 0 rpy=0 0 0, axis 1 0 0, limit lower=-2.0944 upper=0.349066 effort=20 velocity=1
- added joint r_arm_yaw_joint: type revolute, parent r_arm_roll, child r_arm_yaw, origin xyz=0 0 0 rpy=0 0 0, axis 0 0 1, limit lower=-1.5708 upper=1.5708 effort=20 velocity=1
- added joint r_foot_pitch_joint: type continuous, parent r_knee, child r_foot_pitch, origin xyz=0 0 -0.346000000000011 rpy=0 0 0, axis 0 1 0
- added joint r_foot_roll_joint: type continuous, parent r_foot_pitch, child r_foot_roll, origin xyz=0 0 0 rpy=0 0 0, axis -1 0 0
- added joint r_forearm_pitch_joint: type revolute, parent r_arm_yaw, child r_forearm_pitch, origin xyz=0 0 -0.1636 rpy=0 0 0, axis 0 1 0, limit lower=-1.5708 upper=0 effort=20 velocity=1
- added joint r_hand_pitch_joint: type revolute, parent r_hand_yaw, child r_hand_pitch, origin xyz=0 0 0 rpy=0 0 0, axis 0 1 0, limit lower=-1.5708 upper=1.5708 effort=20 velocity=1
- added joint r_hand_roll_joint: type revolute, parent r_hand_pitch, child r_hand_roll, origin xyz=0 0 -0.0590000000076598 rpy=0 0 0, axis 1 0 0, limit lower=-1.5708 upper=1.5708 effort=20 velocity=1
- added joint r_hand_yaw_joint: type revolute, parent r_forearm_pitch, child r_hand_yaw, origin xyz=0 0 -0.132050000118069 rpy=0 0 0, axis 0 0 1, limit lower=-1.5708 upper=1.5708 effort=20 velocity=1
- added joint r_index_distal_finger_joint: type continuous, parent r_index_proximal_finger, child r_index_distal_finger, origin xyz=0.000133519493595612 -0.00243998929947775 -0.0349145904281185 rpy=0 0 0, axis -0.998506141360649 -0.0546395979585212 0
- added joint r_index_proximal_finger_joint: type continuous, parent r_hand_roll, child r_index_proximal_finger, origin xyz=0.0285187933054979 -0.0039487923396026 -0.174730558860479 rpy=0 -0.0311675978215671 0, axis 0.998506141360647 0.0546395979585406 0
- added joint r_knee_joint: type continuous, parent r_leg_pitch, child r_knee, origin xyz=-0.0103901619526017 0 -0.249783995753447 rpy=0 0 0, axis 0 1 0
- added joint r_l_bar_joint: type continuous, parent r_knee, child r_l_bar, origin xyz=0 0.0260000000000006 -0.153 rpy=0 0 0, axis 0 -1 0
- added joint r_l_tendon_joint: type continuous, parent r_l_bar, child r_l_tendon, origin xyz=-0.0579999990740259 0 -1.03629629334412E-05 rpy=0 0 0, axis 0 -1 0
- added joint r_leg_pitch_joint: type continuous, parent r_leg_yaw, child r_leg_pitch, origin xyz=0 -0.0254500000000034 -0.123449999999998 rpy=0 0 0, axis 0 -1 0
- added joint r_leg_roll_joint: type continuous, parent torso, child r_leg_roll, origin xyz=-0.00254758231249268 -0.0870000000000003 -0.0660000000049238 rpy=0 0 0, axis -1 0 0
- added joint r_leg_yaw_joint: type continuous, parent r_leg_roll, child r_leg_yaw, origin xyz=0 0 0 rpy=0 0 0, axis 0 0 1
- added joint r_middle_distal_finger_joint: type continuous, parent r_middle_proximal_finger, child r_middle_distal_finger, origin xyz=0 -0.00292977189725413 -0.0418976901109125 rpy=0 0 0, axis -1 0 0
- added joint r_middle_proximal_finger_joint: type continuous, parent r_hand_roll, child r_middle_proximal_finger, origin xyz=0.00751625831450465 -0.00820381922686125 -0.178435376742697 rpy=0 0 0, axis 1 0 0
- added joint r_pinky_distal_finger_joint: type continuous, parent r_pinky_proximal_finger, child r_pinky_distal_finger, origin xyz=-0.00013921709411558 -0.0024355292668054 -0.0349148795757724 rpy=0 0 0, axis -0.99837030712233 0.0570677654763578 0
- added joint r_pinky_proximal_finger_joint: type continuous, parent r_hand_roll, child r_pinky_proximal_finger, origin xyz=-0.0342146631046227 -0.0036338733880803 -0.17022700803684 rpy=0 0.0659957839625563 0, axis 0.998370307122331 -0.0570677654763477 0
- added joint r_r_bar_joint: type continuous, parent r_knee, child r_r_bar, origin xyz=0 -0.0259999999999875 -0.09 rpy=0 0 0, axis 0 -1 0
- added joint r_r_tendon_joint: type continuous, parent r_r_bar, child r_r_tendon, origin xyz=-0.0579999994737613 0 0 rpy=0 0 0, axis 0 1 0
- added joint r_ring_distal_finger_joint: type continuous, parent r_ring_proximal_finger, child r_ring_distal_finger, origin xyz=-0.000160223392313565 -0.00292798715935183 -0.0418975085136676 rpy=0 0 0, axis -0.996566833460806 -0.0546395979585212 -0.0622017747402293
- added joint r_ring_proximal_finger_joint: type continuous, parent r_hand_roll, child r_ring_proximal_finger, origin xyz=-0.0135862766764854 -0.00807856148813096 -0.176446661066022 rpy=0 0.0311675978215922 0, axis 0.998506141360648 -0.0546395979585354 0
- added joint r_thumb_distal_pitch_joint: type continuous, parent r_thumb_proximal_yaw, child r_thumb_distal_pitch, origin xyz=0.0120000000000024 0.00650000000000001 0.00039999999999929 rpy=0 0 0, axis 0 -1 0
- added joint r_thumb_proximal_yaw_joint: type continuous, parent r_hand_roll, child r_thumb_proximal_yaw, origin xyz=0.0240162583145044 0.0216278329431261 -0.110700000402968 rpy=0 0 0, axis 0 0 1

File: src/robot_model_pkg/biped_s4/urdf/biped_s4_orin.urdf (robot description, URDF)
Before this commit: robot biped_s4, 57 links, 56 joints
Links:
- added link head_camera; visual sphere radius=0.001
- added link l_hand_end_virtual; visual sphere radius=0.001
- added link r_hand_end_virtual; visual sphere radius=0.001
- added link torso_camera; visual sphere radius=0.001
Joints:
- added joint head_camera: type fixed, parent head_pitch, child head_camera, origin xyz=0.082 0.0175 0.05449 rpy=0 0.6105555 0
- added joint l_hand_end_virtual: type fixed, parent l_hand_roll, child l_hand_end_virtual, origin xyz=0 0 -0.1545 rpy=0 0 0
- added joint r_hand_end_virtual: type fixed, parent r_hand_roll, child r_hand_end_virtual, origin xyz=0 0 -0.1545 rpy=0 0 0
- added joint torso_camera: type fixed, parent torso, child torso_camera, origin xyz=0.11416 0.0175 0.28459 rpy=0 0.71522222 0
- joint l_arm_pitch: limit (none) -> lower=-3.14159 upper=0.523599 effort=20 velocity=1; type continuous -> revolute
- joint l_arm_roll: limit (none) -> lower=-0.349066 upper=2.0944 effort=20 velocity=1; type continuous -> revolute
- joint l_arm_yaw: limit (none) -> lower=-1.5708 upper=1.5708 effort=20 velocity=1; type continuous -> revolute
- joint l_forearm_pitch: limit (none) -> lower=-1.5708 upper=0 effort=20 velocity=1; type continuous -> revolute
- joint l_hand_pitch: limit (none) -> lower=-1.5708 upper=1.5708 effort=20 velocity=1; type continuous -> revolute
- joint l_hand_roll: limit (none) -> lower=-1.5708 upper=1.5708 effort=20 velocity=1; type continuous -> revolute
- joint l_hand_yaw: limit (none) -> lower=-1.5708 upper=1.5708 effort=20 velocity=1; type continuous -> revolute
- joint r_arm_pitch: limit (none) -> lower=-3.14159 upper=0.523599 effort=20 velocity=1; type continuous -> revolute
- joint r_arm_roll: limit (none) -> lower=-2.0944 upper=0.349066 effort=20 velocity=1; type continuous -> revolute
- joint r_arm_yaw: limit (none) -> lower=-1.5708 upper=1.5708 effort=20 velocity=1; type continuous -> revolute
- joint r_forearm_pitch: limit (none) -> lower=-1.5708 upper=0 effort=20 velocity=1; type continuous -> revolute
- joint r_hand_pitch: limit (none) -> lower=-1.5708 upper=1.5708 effort=20 velocity=1; type continuous -> revolute
- joint r_hand_roll: limit (none) -> lower=-1.5708 upper=1.5708 effort=20 velocity=1; type continuous -> revolute
- joint r_hand_yaw: limit (none) -> lower=-1.5708 upper=1.5708 effort=20 velocity=1; type continuous -> revolute
